Commit message: Add gripper fix

File: src/robot_arm_moveit/config/gazebo_rob_manip_2.urdf (robot description, URDF)
Before this commit: robot rob_manip_2, 9 links, 8 joints
Links:
- added link left_gripper, mass 0.1; collision box size=0.02 0.02 0.07; visual box size=0.02 0.02 0.07
- added link right_gripper, mass 0.1; collision box size=0.02 0.02 0.07; visual box size=0.02 0.02 0.07
- link hand: geometry collision box size=0.05 0.12 0.02; visual box size=0.03 0.12 0.02
Joints:
- added joint gripper_joint_left: type prismatic, parent hand, child left_gripper, origin xyz=0 0.05 0.0175 rpy=0 0 0, axis 0 -1 0, limit lower=0.0 upper=0.04 effort=1000 velocity=0.1
- added joint gripper_joint_right: type prismatic, parent hand, child right_gripper, origin xyz=0 -0.05 0.0175 rpy=0 0 0, axis 0 1 0, limit lower=0.0 upper=0.04 effort=1000 velocity=0.1

File: src/robot_arm_moveit/urdf/rob_manip_2.urdf (robot description, URDF)
Before this commit: robot rob_manip_2, 9 links, 8 joints
Links:
- added link left_gripper, mass 0.1; collision box size=0.02 0.02 0.07; visual box size=0.02 0.02 0.07
- added link right_gripper, mass 0.1; collision box size=0.02 0.02 0.07; visual box size=0.02 0.02 0.07
- link hand: geometry collision box size=0.05 0.12 0.02; visual box size=0.03 0.12 0.02
Joints:
- added joint gripper_joint_left: type prismatic, parent hand, child left_gripper, origin xyz=0 0.05 0.0175 rpy=0 0 0, axis 0 -1 0, limit lower=0.0 upper=0.04 effort=1000 velocity=0.1
- added joint gripper_joint_right: type prismatic, parent hand, child right_gripper, origin xyz=0 -0.05 0.0175 rpy=0 0 0, axis 0 1 0, limit lower=0.0 upper=0.04 effort=1000 velocity=0.1
